File: Connectors.kicad_sch (KiCad schematic)
At the start: 5 parts, among them U4 PESD4USB5U-TTSX, U5 PESD4USB5U-TTSX, U7 PESD4USB5U-TTSX, U8 PESD4USB5U-TTSX

Commit message: initial
Parts:
- removed J4: (no value), X3.0CH-Library:X3.0CH-Master, symbol X3.0CH-Library:X3.0-CH
- added J1, J2, J3: Conn_02x10_Odd_Even, X3.0CH-Library:Hanxia_HX_PM1.0-2x10P_ZC, symbol Connector_Generic:Conn_02x10_Odd_Even
Connections:
- net +3.3V: now also J1.3 (Pin_3)
- net +5V: now also J1.1 (Pin_1)
- net CURR1 FILTERED: now also J2.13 (Pin_13)
- net CURR2 FILTERED: now also J2.3 (Pin_3)
- net CURR3 FILTERED: now also J1.13 (Pin_13)
- net ESP-RX: now also J3.5 (Pin_5)
- net ESP-TX: now also J3.3 (Pin_3)
- net GND: now also J1.10 (Pin_10), J1.12 (Pin_12), J1.14 (Pin_14), J1.16 (Pin_16), J1.18 (Pin_18), J1.2 (Pin_2), J1.20 (Pin_20), J1.8 (Pin_8), J2.10 (Pin_10), J2.12 (Pin_12), J2.14 (Pin_14), J2.16 (Pin_16), J2.2 (Pin_2), J2.4 (Pin_4), J2.6 (Pin_6), J2.8 (Pin_8), J3.1 (Pin_1), J3.10 (Pin_10), J3.20 (Pin_20)
- net H1: now also J2.9 (Pin_9)
- net H2: now also J1.19 (Pin_19)
- net H3: now also J1.9 (Pin_9)
- net HALL-VOLTAGE: now also J3.7 (Pin_7)
- net HALL1 IN: now also J3.9 (Pin_9)
- net HALL2 IN: now also J3.11 (Pin_11)
- net HALL3 IN: now also J3.12 (Pin_12)
- net I2C2 SCL/USART3 TX: now also J3.17 (Pin_17)
- net I2C2 SDA/USART3 RX: now also J3.16 (Pin_16)
- net IN V: now also J1.4 (Pin_4)
- net IN-CANH: now also J3.6 (Pin_6)
- net IN-CANL: now also J3.8 (Pin_8)
- net L1: now also J2.11 (Pin_11)
- net L2: now also J2.1 (Pin_1)
- net L3: now also J1.11 (Pin_11)
- net MOSTEMP1: now also J2.7 (Pin_7)
- net MOSTEMP2: now also J1.17 (Pin_17)
- net MOSTEMP3: now also J1.7 (Pin_7)
- net NRST: now also J3.15 (Pin_15)
- net POWER STAGE DISABLE: now also J1.5 (Pin_5)
- net POWER STAGE LOCKOUT: now also J1.6 (Pin_6)
- net SERVO: now also J3.13 (Pin_13)
- net SPI1-MISO-ADC2: now also J2.19 (Pin_19)
- net SPI1-MOSI: now also J2.17 (Pin_17)
- net SPI1-NSS: now also J3.4 (Pin_4)
- net SPI1-SCK-ADC: now also J3.2 (Pin_2)
- net SWCLK: now also J3.19 (Pin_19)
- net SWDIO: now also J3.18 (Pin_18)
- net TEMPMOTOR IN: now also J3.14 (Pin_14)
- net USBD+: now also J2.20 (Pin_20)
- net USBD-: now also J2.18 (Pin_18)
- net VSENSE1: now also J2.15 (Pin_15)
- net VSENSE2: now also J2.5 (Pin_5)
- net VSENSE3: now also J1.15 (Pin_15)
Other:
- note added: "41 non-ground signals and 19 GND contacts. Right-angle male headers on the power PCB."
- note added: "Columns 4-8: phase 3 | 9-13: phase 2 | 14-18: phase 1. Opposite phase contacts: GND."
- note added: "ESD protection retained on the original nets"
- note added: "F.Cu view: J1 -> J2 -> J3. Active signal order retained; J3 grounds at pins 1, 10, 20."
- note added: "J1 + J2 + J3: 60 contacts, three 2x10 straight sockets, 1.00 mm pitch."
- moved on the sheet: U4, U5, U7, U8

Commit message: pre-full-route
Connections:
- net HALL-VOLTAGE is gone; now on net GND: J3.7 (Pin_7)
- net ESP-RX: now also J3.20 (Pin_20), U5.4, U5.7; no longer J3.5 (Pin_5), U7.5, U7.6
- net ESP-TX: now also J3.19 (Pin_19), U5.2, U5.9; no longer J3.3 (Pin_3), U7.4, U7.7
- net GND: now also J3.18 (Pin_18), J3.4 (Pin_4); no longer J3.1 (Pin_1), J3.20 (Pin_20)
- net HALL3 IN: now also J3.13 (Pin_13); no longer J3.12 (Pin_12)
- net I2C2 SCL/USART3 TX: now also J3.8 (Pin_8), U7.1, U7.10; no longer J3.17 (Pin_17), U5.5, U5.6
- net I2C2 SDA/USART3 RX: now also J3.6 (Pin_6), U7.2, U7.9; no longer J3.16 (Pin_16), U5.4, U5.7
- net IN-CANH: now also J3.16 (Pin_16); no longer J3.6 (Pin_6)
- net IN-CANL: now also J3.14 (Pin_14); no longer J3.8 (Pin_8)
- net NRST: now also J3.17 (Pin_17); no longer J3.15 (Pin_15)
- net SERVO: now also J3.12 (Pin_12), U5.5, U5.6; no longer J3.13 (Pin_13), U5.2, U5.9
- net SPI1-MISO-ADC2: now also J2.20 (Pin_20), U4.4, U4.7; no longer J2.19 (Pin_19), U4.2, U4.9
- net SPI1-MOSI: now also J2.18 (Pin_18), U4.5, U4.6; no longer J2.17 (Pin_17), U4.1, U4.10
- net SPI1-NSS: now also J2.17 (Pin_17), U4.1, U4.10; no longer J3.4 (Pin_4), U4.5, U4.6
- net SPI1-SCK-ADC: now also J2.19 (Pin_19), U4.2, U4.9; no longer J3.2 (Pin_2), U4.4, U4.7
- net SWCLK: now also J3.5 (Pin_5), U7.5, U7.6; no longer J3.19 (Pin_19), U7.2, U7.9
- net SWDIO: now also J3.3 (Pin_3), U7.4, U7.7; no longer J3.18 (Pin_18), U7.1, U7.10
- net TEMPMOTOR IN: now also J3.15 (Pin_15); no longer J3.14 (Pin_14)
- net USBD+: now also J3.1 (Pin_1); no longer J2.20 (Pin_20)
- net USBD-: now also J3.2 (Pin_2); no longer J2.18 (Pin_18)
Other:
- moved on the sheet: U7

Commit message: initial
Connections:
- net CURR1 FILTERED renamed CURR1-FILTERED
- net CURR2 FILTERED renamed CURR2-FILTERED
- net CURR3 FILTERED renamed CURR3-FILTERED
- net HALL1 IN renamed TEMPMOTOR-IN
- net TEMPMOTOR-IN: now also J3.15 (Pin_15); no longer J3.9 (Pin_9)
- net HALL2 IN renamed HALL3-IN
- net HALL3-IN: now also J3.13 (Pin_13); no longer J3.11 (Pin_11)
- net HALL3 IN renamed HALL2-IN
- net HALL2-IN: now also J3.11 (Pin_11); no longer J3.13 (Pin_13)
- net I2C2 SCL/USART3 TX renamed I2C2-SCL/USART3-TX
- net I2C2 SDA/USART3 RX renamed I2C2-SDA/USART3-RX
- net IN V renamed IN-V
- net POWER STAGE DISABLE renamed POWER-STAGE-DISABLE
- net POWER STAGE LOCKOUT renamed POWER-STAGE-LOCKOUT
- net TEMPMOTOR IN renamed HALL1-IN
- net HALL1-IN: now also J3.9 (Pin_9); no longer J3.15 (Pin_15)
Other:
- moved on the sheet: U4
