File: Filters.kicad_sch (KiCad schematic)
At the start: 11 parts

Commit message: pre-full-route
Parts:
- removed JP3: VSel, X3.0CH-Library:SolderJumper-3-0.5-Small, symbol Jumper:Jumper_3_Bridged12

Commit message: initial
Parts:
- removed C30: 1n, Capacitor_SMD:C_0402_1005Metric, symbol Device:C
Connections:
- net HALL1 IN renamed HALL1-IN
- net HALL2 IN renamed HALL2-IN
- net HALL3 IN renamed HALL3-IN
- net PHASE FILTER ENABLE1 renamed PHASE-FILTER-ENABLE1
- net PHASE FILTER ENABLE2 renamed PHASE-FILTER-ENABLE2
- net PHASE FILTER ENABLE3 renamed PHASE-FILTER-ENABLE3
- net TEMPMOTOR IN renamed TEMPMOTOR-IN
Other:
- note removed: "Input Voltage Filter"
