File: GigaControl.kicad_pcb (KiCad board)
At the start: 6 copper layers, 40 x 20 mm, 49 parts, among them U1 LSM6DS3TR-C, U2 SIT3051, U3 REF3033AIDBZR, U4 PESD4USB5U-TTSX, U5 PESD4USB5U-TTSX, U6 STM32F405RGT6, U7 PESD4USB5U-TTSX, U8 PESD4USB5U-TTSX, Y1 SX2M8.000M20F30TNN

Commit message: initial
Parts:
- removed J4: ~, X3.0CH-Library:X3.0CH-Master
- removed REF** (x2): PinHeader_2x15_P1.27mm_Vertical, Connector_PinHeader_1.27mm:PinHeader_2x15_P1.27mm_Vertical
- added J1: Conn_02x10_Odd_Even, X3.0CH-Library:Hanxia_HX_PM1.0-2x10P_ZC, F.Cu at (138.6, 87.7)
- added J2: Conn_02x10_Odd_Even, X3.0CH-Library:Hanxia_HX_PM1.0-2x10P_ZC, F.Cu at (150.1, 87.7)
- added J3: Conn_02x10_Odd_Even, X3.0CH-Library:Hanxia_HX_PM1.0-2x10P_ZC, F.Cu at (161.6, 87.7)
- moved C27 4.74 mm to (159.1, 94.1)
- moved C3 4.74 mm to (156.2, 105.6)
- moved C47 4.74 mm to (158.1, 103.3)
- moved R3 4.74 mm to (160.2, 103.3)
- moved U5 4.74 mm to (154.2, 106.6)
- moved C16 4.74 mm to (143.6, 102.5)
- moved C18 4.74 mm to (155.1, 90.2)
- moved C2 4.74 mm to (143.6, 106.9)
- moved C20 4.74 mm to (144.6, 102.5)
- moved C28 4.74 mm to (157.7, 92.7)
- moved D1 4.74 mm to (144.2, 95.5)
- moved D2 4.74 mm to (161.7, 105.5)
- moved R1 4.74 mm to (148.2, 105.7)
- moved R11 4.74 mm to (144.1, 97.7)
- moved R13 4.74 mm to (146.2, 89.7)
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Other:
- board size 40 x 20 mm -> 34.4 x 20 mm

Commit message: initial
Parts:
- added H1: MountingHole_3.2mm_M3, MountingHole:MountingHole_3.2mm_M3, F.Cu at (140.0, 103.0)
- added H2: MountingHole_3.2mm_M3, MountingHole:MountingHole_3.2mm_M3, F.Cu at (169.2, 103.0)
- moved D2 26.3 mm to (140.0, 90.6)
- moved R12 26.3 mm to (139.8, 92.7)
- moved U5 22.6 mm to (169.7, 90.1)
- moved U7 22.6 mm to (166.3, 90.1)
- moved U8 22.0 mm to (165.9, 97.9)
- moved C26 16.5 mm to (143.3, 93.1)
- moved C30 16.5 mm to (143.3, 95.1)
- moved C27 16.5 mm to (142.9, 91.5)
- moved C28 16.5 mm to (141.5, 90.1)
- moved C3 15.6 mm to (165.3, 92.9)
- moved R3 15.0 mm to (170.2, 92.1)
- moved U2 15.0 mm to (168.8, 94.4)
- moved C2 9.74 mm to (138.8, 98.5)
- moved U1 9.74 mm to (140.8, 97.5)
- moved R1 9.74 mm to (143.4, 97.2)
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Routing:
- net +5V: track 39.5 -> 20.0 mm, vias 3 -> 2
- net SPI1-MOSI: track 13.1 -> 23.6 mm
- net VSENSE2: track 9.60 -> 18.4 mm
- net CURR1 FILTERED: track 11.1 -> 17.4 mm
- net VSENSE3: track 12.7 -> 18.9 mm
- net CURR3 FILTERED: track 15.8 -> 21.0 mm
- net H1: track 19.2 -> 24.2 mm
- net H3: track 13.1 -> 18.1 mm
- net L3: track 9.42 -> 14.4 mm
- net MOSTEMP1: track 3.79 -> 8.58 mm
- net MOSTEMP2: track 6.07 -> 10.8 mm
- net RESERVED2: track 9.56 -> 4.90 mm
- net RESERVED3: track 10.1 -> 5.59 mm
- net H2: track 13.2 -> 17.7 mm
- net MOSTEMP3: track 10.4 -> 14.5 mm
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
Commit message: pre-move
Parts:
- moved C28 26.9 mm to (167.4, 97.4), turned to -90 degrees
- moved C27 23.2 mm to (162.6, 103.7)
- moved JP3 19.6 mm to (165.4, 95.0)
- moved C26 18.3 mm to (161.4, 95.7)
- moved C1 11.4 mm to (159.0, 104.6), turned to 0 degrees
- moved R4 8.20 mm to (171.0, 97.0), turned to -90 degrees
- moved D1 7.74 mm to (139.8, 91.0), turned to 180 degrees
- moved R11 7.65 mm to (142.3, 91.0)
- moved C2 4.98 mm to (141.1, 94.1), turned to 0 degrees
- moved C30 2.57 mm to (144.3, 92.7)
- moved R12 2.49 mm to (142.3, 92.5), turned to 0 degrees
- moved R2 2.09 mm to (141.3, 98.7), turned to 90 degrees
- moved D2 1.98 mm to (139.8, 92.6), turned to 180 degrees
- moved U1 1.94 mm to (142.1, 96.1), turned to 180 degrees
- moved R1 1.76 mm to (142.3, 98.7), turned to 90 degrees
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Routing:
- net IN-CANH: track 10.3 -> 6.85 mm
- net VSENSE2: track 18.4 -> 15.1 mm
- net +3.3V: track 72.0 -> 71.0 mm
- net IN-CANL: track 9.30 -> 8.67 mm
- net GND: vias 58 -> 57

Commit message: pre-full-route
Parts:
- removed JP3: VSel, X3.0CH-Library:SolderJumper-3-0.5-Small
- H1, H2: value MountingHole_3.2mm_M3 -> MountingHole; footprint MountingHole:MountingHole_3.2mm_M3 -> MountingHole:MountingHole_3.2mm_M3_DIN965
- moved H1 29.2 mm to (169.2, 103.0)
- moved H2 29.2 mm to (140.0, 103.0)
- moved U3 23.2 mm to (139.3, 95.7), turned to -90 degrees
- moved C5 21.8 mm to (139.1, 98.2), turned to 0 degrees
- moved C1 18.8 mm to (141.1, 98.7), turned to -90 degrees
- moved C27 9.04 mm to (161.4, 94.7), turned to 0 degrees
- moved U8 7.54 mm to (166.5, 90.5), turned to -90 degrees
- moved C28 7.02 mm to (161.4, 93.7), turned to 0 degrees
- moved R15 4.84 mm to (145.9, 97.7)
- moved R16 4.84 mm to (145.9, 96.7)
- moved R17 4.84 mm to (145.9, 95.7)
- moved U4 4.12 mm to (160.3, 90.5), turned to 90 degrees
- moved C3 3.04 mm to (165.9, 95.9)
- moved C17 2.64 mm to (159.0, 103.8), turned to 0 degrees
- moved U7 2.10 mm to (163.4, 90.5)
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Connections:
- J2 pad 17: SPI1-MOSI -> SPI1-NSS
- J2 pad 18: USBD- -> SPI1-MOSI
- J2 pad 19: SPI1-MISO-ADC2 -> SPI1-SCK-ADC
- J2 pad 20: USBD+ -> SPI1-MISO-ADC2
- J3 pad 1: GND -> USBD+
- J3 pad 12: HALL3 IN -> SERVO
- J3 pad 13: SERVO -> HALL3 IN
- J3 pad 14: TEMPMOTOR IN -> IN-CANL
- J3 pad 15: NRST -> TEMPMOTOR IN
- J3 pad 16: I2C2 SDA/USART3 RX -> IN-CANH
- J3 pad 17: I2C2 SCL/USART3 TX -> NRST
- J3 pad 18: SWDIO -> GND
- J3 pad 19: SWCLK -> ESP-TX
- J3 pad 2: SPI1-SCK-ADC -> USBD-
- J3 pad 20: GND -> ESP-RX
- J3 pad 3: ESP-TX -> SWDIO
- J3 pad 4: SPI1-NSS -> GND
- J3 pad 5: ESP-RX -> SWCLK
- J3 pad 6: IN-CANH -> I2C2 SDA/USART3 RX
- J3 pad 7: HALL-VOLTAGE -> GND
- J3 pad 8: IN-CANL -> I2C2 SCL/USART3 TX
- U4 pad 1: SPI1-MOSI -> SPI1-NSS
- U4 pad 10: SPI1-MOSI -> SPI1-NSS
- U4 pad 2: SPI1-MISO-ADC2 -> SPI1-SCK-ADC
- U4 pad 4: SPI1-SCK-ADC -> SPI1-MISO-ADC2
- U4 pad 5: SPI1-NSS -> SPI1-MOSI
- U4 pad 6: SPI1-NSS -> SPI1-MOSI
- U4 pad 7: SPI1-SCK-ADC -> SPI1-MISO-ADC2
- U4 pad 9: SPI1-MISO-ADC2 -> SPI1-SCK-ADC
- U5 pad 2: SERVO -> ESP-TX
- U5 pad 4: I2C2 SDA/USART3 RX -> ESP-RX
- U5 pad 5: I2C2 SCL/USART3 TX -> SERVO
- U5 pad 6: I2C2 SCL/USART3 TX -> SERVO
- U5 pad 7: I2C2 SDA/USART3 RX -> ESP-RX
- U5 pad 9: SERVO -> ESP-TX
- U7 pad 1: SWDIO -> I2C2 SCL/USART3 TX
- U7 pad 10: SWDIO -> I2C2 SCL/USART3 TX
- U7 pad 2: SWCLK -> I2C2 SDA/USART3 RX
- U7 pad 4: ESP-TX -> SWDIO
- U7 pad 5: ESP-RX -> SWCLK
- U7 pad 6: ESP-RX -> SWCLK
- U7 pad 7: ESP-TX -> SWDIO
- U7 pad 9: SWCLK -> I2C2 SDA/USART3 RX
Routing:
- net SERVO: track 4.93 -> 34.8 mm, vias 0 -> 2
- net ESP-RX: track 5.40 -> 31.4 mm, vias 0 -> 2
- net ESP-TX: track 6.97 -> 30.0 mm, vias 0 -> 2
- net SWCLK: track 5.57 -> 27.3 mm, vias 0 -> 2
- net HALL3 IN: track 10.5 -> 29.0 mm
- net SWDIO: track 8.70 -> 26.6 mm
- net HALL2 IN: track 11.1 -> 27.6 mm
- net USBD-: track 18.0 -> 33.7 mm
- net HALL1 IN: track 11.3 -> 27.0 mm
- net USBD+: track 18.0 -> 33.7 mm
- net IN V: track 18.0 -> 32.3 mm, vias 1 -> 4
- net +3.3REF: track 12.0 -> 25.9 mm, vias 0 -> 2
- net LED FAULT: track 14.3 -> 0.88 mm, vias 2 -> 1
- net POWER STAGE LOCKOUT: track 5.25 -> 18.2 mm
- net TEMPMOTOR IN: track 16.7 -> 28.9 mm
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
Commit message: full-route
Parts:
- added TP1: TestPoint, TestPoint:TestPoint_Pad_D1.0mm, F.Cu at (147.8, 104.0)
- added TP2: TestPoint, TestPoint:TestPoint_Pad_D1.0mm, F.Cu at (145.7, 104.0)
- added TP3: TestPoint, TestPoint:TestPoint_Pad_D1.0mm, F.Cu at (163.5, 104.2)
- moved C1 5.82 mm to (143.5, 93.4), turned to 90 degrees
- moved C5 4.90 mm to (140.1, 93.4)
- moved C30 3.18 mm to (144.1, 90.9), turned to -90 degrees
- moved R2 2.60 mm to (144.6, 99.7), turned to 180 degrees
- moved R4 2.32 mm to (170.7, 96.3), turned to 90 degrees
- moved R3 1.91 mm to (168.3, 93.8)
- moved R1 1.40 mm to (144.6, 98.7), turned to 180 degrees
- moved C3 0.98 mm to (165.0, 96.3)
- moved U2 0.98 mm to (167.9, 96.3)
- moved U3 0.30 mm to (139.3, 96.0)
- moved H1 0.10 mm to (169.3, 103.0)
- moved C16 0.10 mm to (145.6, 100.8)
- moved H2 0.10 mm to (139.9, 103.0)
Routing:
- net LED RUN: track 1.45 -> 24.6 mm, vias 1 -> 2
- net LED FAULT: track 0.88 -> 22.7 mm, vias 1 -> 2
- net +3.3V: track 70.6 -> 90.5 mm, vias 7 -> 4
- net IMU SDA: track 4.27 -> 20.5 mm
- net CAN TX: track 3.58 -> 18.9 mm
- net IMU SCL: track 5.44 -> 20.4 mm
- net CAN RX: track 4.18 -> 17.3 mm, vias 1 -> 2
- net RESERVED3: track 0.00 -> 11.4 mm
- net RESERVED2: track 0.00 -> 8.58 mm
- net IN-CANL: track 10.8 -> 16.6 mm
- net IN-CANH: track 9.14 -> 13.9 mm, vias 0 -> 1
- net GND: track 9.79 -> 13.4 mm, vias 39 -> 56
- net RESERVED1: track 0.72 -> 3.74 mm
- net Net-(D2-K): track 0.00 -> 1.37 mm
- net Net-(U2-S): track 0.49 -> 1.80 mm
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Other:
- board text added: "X3.0 SLOT"
- board text removed: "3.3V"
- board text removed: "5V"
- board text removed: "CAN-H"
- board text removed: "CAN-L"
- board text removed: "CLK"
- board text removed: "DIO"
- board text removed: "GND"
- board text removed: "HALL-VCC"
- board text removed: "HALL1"
- board text removed: "HALL2"
- board text removed: "HALL3"
- board text removed: "IN-V"
- board text removed: "MISO/ADC2"
- board text removed: "MOSI"
- board text removed: "NRST"
- board text removed: "NSS"
- board text removed: "R1"
- board text removed: "R2"
- board text removed: "R3"
- board text removed: "SCK/ADC1"
- board text removed: "SERVO"
- board text removed: "T-MOT"
- board text removed: "U1-RX"
- board text removed: "U1-TX"
- board text removed: "U3-RX"
- board text removed: "U3-TX"
- board text removed: "USB+"
- board text removed: "USB-"
- board text removed: "X3.0 CH"

Commit message: initial
Parts:
- added JP1: VREF->3V3, Jumper:SolderJumper-2_P1.3mm_Open_RoundedPad1.0x1.5mm, F.Cu at (164.0, 98.2)
- moved R10 3.83 mm to (163.9, 96.0), turned to 90 degrees
- moved C25 2.56 mm to (164.5, 94.5), turned to 0 degrees
- moved C3 0.30 mm to (165.0, 96.0)
- turned U8 to 90 degrees
Connections:
- net CAN RX renamed /CAN-RX
- net CAN TX renamed /CAN-TX
- net CURR1 FILTERED renamed /CURR1-FILTERED
- net CURR2 FILTERED renamed /CURR2-FILTERED
- net CURR3 FILTERED renamed /CURR3-FILTERED
- net ESP-RX renamed /ESP-RX
- net ESP-TX renamed /ESP-TX
- net H1 renamed /H1
- net H2 renamed /H2
- net H3 renamed /H3
- net HALL1 renamed /HALL1
- net HALL2 renamed /HALL2
- net HALL3 renamed /HALL3
- net I2C2 SCL/USART3 TX renamed /I2C2-SCL/USART3-TX
- net I2C2 SDA/USART3 RX renamed /I2C2-SDA/USART3-RX
- net IMU SCL renamed /IMU-SCL
- net IMU SDA renamed /IMU-SDA
- net IN-CANH renamed /IN-CANH
- net IN-CANL renamed /IN-CANL
- net L1 renamed /L1
- net L2 renamed /L2
- net L3 renamed /L3
- net LED FAULT renamed /MCU/LED-FAULT
- net LED RUN renamed /MCU/LED-RUN
- net MOSTEMP1 renamed /MOSTEMP1
- net MOSTEMP2 renamed /MOSTEMP2
- net MOSTEMP3 renamed /MOSTEMP3
- net NRST renamed /NRST
- net PHASE FILTER ENABLE1 renamed /PHASE-FILTER-ENABLE1
- net PHASE FILTER ENABLE2 renamed /PHASE-FILTER-ENABLE2
- net PHASE FILTER ENABLE3 renamed /PHASE-FILTER-ENABLE3
- net POWER STAGE DISABLE renamed /POWER-STAGE-DISABLE
- net POWER STAGE LOCKOUT renamed /POWER-STAGE-LOCKOUT
- net RESERVED1 renamed /MCU/RESERVED1
- net RESERVED2 renamed /MCU/RESERVED2
- net RESERVED3 renamed /MCU/RESERVED3
- net SERVO renamed /SERVO
- net SPI1-MISO-ADC2 renamed /SPI1-MISO-ADC2
- net SPI1-MOSI renamed /SPI1-MOSI
- net SPI1-NSS renamed /SPI1-NSS
- net SPI1-SCK-ADC renamed /SPI1-SCK-ADC
- net SWCLK renamed /SWCLK
- net SWDIO renamed /SWDIO
- net TEMPMOTOR renamed /TEMPMOTOR
- net USBD+ renamed /USBD+
- net USBD- renamed /USBD-
- net VSENSE1 renamed /VSENSE1
- net VSENSE2 renamed /VSENSE2
- net VSENSE3 renamed /VSENSE3
- C30 pad 1: IN V -> /IN-V
- J1 pad 4: IN V -> +3.3REF
- J1 pad 8: GND -> /IN-V
- J3 pad 11: HALL2 IN -> /HALL2-IN
- J3 pad 13: HALL3 IN -> /HALL3-IN
- J3 pad 15: TEMPMOTOR IN -> /TEMPMOTOR-IN
- J3 pad 9: HALL1 IN -> /HALL1-IN
- R13 pad 1: TEMPMOTOR IN -> /TEMPMOTOR-IN
- R14 pad 1: TEMPMOTOR IN -> /TEMPMOTOR-IN
- R15 pad 2: HALL3 IN -> /HALL3-IN
- R16 pad 2: HALL2 IN -> /HALL2-IN
- R17 pad 2: HALL1 IN -> /HALL1-IN
- U6 pad 11: IN V -> /IN-V
- U8 pad 1: TEMPMOTOR IN -> /HALL1-IN
- U8 pad 10: TEMPMOTOR IN -> /HALL1-IN
- U8 pad 2: HALL3 IN -> /HALL2-IN
- U8 pad 4: HALL2 IN -> /HALL3-IN
- U8 pad 5: HALL1 IN -> /TEMPMOTOR-IN
- U8 pad 6: HALL1 IN -> /TEMPMOTOR-IN
- U8 pad 7: HALL2 IN -> /HALL3-IN
- U8 pad 9: HALL3 IN -> /HALL2-IN
Routing:
- net /TEMPMOTOR-IN: track 0.00 -> 35.3 mm, vias 0 -> 2
- net /IN-V: track 0.00 -> 34.1 mm, vias 0 -> 3
- net IN V: track 32.4 -> 0.00 mm, vias 4 -> 0
- net TEMPMOTOR IN: track 30.0 -> 0.00 mm, vias 2 -> 0
- net HALL3 IN: track 28.9 -> 0.00 mm, vias 2 -> 0
- net /HALL3-IN: track 0.00 -> 28.9 mm, vias 0 -> 2
- net HALL2 IN: track 27.6 -> 0.00 mm, vias 2 -> 0
- net /HALL2-IN: track 0.00 -> 27.6 mm, vias 0 -> 2
- net HALL1 IN: track 27.0 -> 0.00 mm, vias 2 -> 0
- net /HALL1-IN: track 0.00 -> 27.0 mm, vias 0 -> 2
- net +3.3REF: track 25.8 -> 38.8 mm, vias 2 -> 3
- net +3.3V: track 90.5 -> 88.7 mm
- net GND: track 13.4 -> 14.6 mm, vias 56 -> 64
- net /L1: track 18.5 -> 17.9 mm, vias 2 -> 1
- net /NRST: track 17.2 -> 17.4 mm, vias 0 -> 2
Other:
- board text added: "3.3R"
- board text added: "R1"
- board text added: "R2"
- board text added: "R3"
