File: GigaControl.kicad_sch (KiCad schematic)
At the start: 0 parts

Commit message: pre-full-route
Parts:
- added H1, H2: MountingHole, MountingHole:MountingHole_3.2mm_M3_DIN965, symbol Mechanical:MountingHole
Changed lines of the file:
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@@
 		(rev "V1.1.0")
+	)
+	(symbol
+		(lib_id "Mechanical:MountingHole")
+		(at 222.25 36.83 0)
+		(unit 1)
+		(body_style 1)
+		(exclude_from_sim no)
+		(in_bom no)
+		(on_board yes)
+		(in_pos_files yes)
+		(dnp no)
+		(fields_autoplaced yes)
+		(property "Reference" "H1"
+			(at 224.79 35.5599 0)
+			(show_name no)
+			(do_not_autoplace no)
+			(effects
+				(font
+					(size 1.27 1.27)
+				)
+				(justify left)
+			)
+		)
+		(property "Value" "MountingHole"
+			(at 224.79 38.0999 0)
+			(show_name no)
+			(do_not_autoplace no)
+			(effects
+				(font
+					(size 1.27 1.27)
+				)
+				(justify left)
+			)
+		)
+		(property "Footprint" "MountingHole:MountingHole_3.2mm_M3_DIN965"
+			(at 222.25 36.83 0)
+			(hide yes)
+			(show_name no)
+			(do_not_autoplace no)
+			(effects
+				(font
+					(size 1.27 1.27)
+				)
+			)
+		)
+		(property "Datasheet" ""
+			(at 222.25 36.83 0)
+			(hide yes)
+			(show_name no)
+			(do_not_autoplace no)
+			(effects
+				(font
+					(size 1.27 1.27)
+				)
+			)
+		)
+		(property "Description" "Mounting Hole without connection"
+			(at 222.25 36.83 0)
+			(hide yes)
+			(show_name no)
+			(do_not_autoplace no)
+			(effects
+				(font
+					(size 1.27 1.27)
+				)
+			)
+		)
+		(instances
+			(project "GigaControl"
+				(path "/0468a8f0-6992-48fb-8a0a-32fabb565718"
+					(reference "H1")
+					(unit 1)
+				)
+			)
+		)
+	)
+	(symbol
+		(lib_id "Mechanical:MountingHole")
+		(at 222.25 43.18 0)
+		(unit 1)
+		(body_style 1)
+		(exclude_from_sim no)
+		(in_bom no)
+		(on_board yes)
+		(in_pos_files yes)
+		(dnp no)
+		(fields_autoplaced yes)
+		(property "Reference" "H2"
+			(at 224.79 41.9099 0)
+			(show_name no)
+			(do_not_autoplace no)
+			(effects
+				(font
+					(size 1.27 1.27)
+				)
+				(justify left)
+			)
+		)
+		(property "Value" "MountingHole"
+			(at 224.79 44.4499 0)
+			(show_name no)
+			(do_not_autoplace no)
+			(effects
+				(font
+					(size 1.27 1.27)
+				)
+				(justify left)
+			)
+		)
+		(property "Footprint" "MountingHole:MountingHole_3.2mm_M3_DIN965"
+			(at 222.25 43.18 0)
+			(hide yes)
+			(show_name no)
+			(do_not_autoplace no)
+			(effects
+				(font
+					(size 1.27 1.27)
+				)
+			)
+		)
+		(property "Datasheet" ""
+			(at 222.25 43.18 0)
+			(hide yes)
+			(show_name no)
+			(do_not_autoplace no)
+			(effects
+				(font
+					(size 1.27 1.27)
+				)
+			)
+		)
+		(property "Description" "Mounting Hole without connection"
+			(at 222.25 43.18 0)
+			(hide yes)
+			(show_name no)
+			(do_not_autoplace no)
+			(effects
+				(font
+					(size 1.27 1.27)
+				)
+			)
+		)
+		(instances
+			(project "GigaControl"
+				(path "/0468a8f0-6992-48fb-8a0a-32fabb565718"
+					(reference "H2")
+					(unit 1)
+				)
+			)
+		)
 	)
 	(sheet

Commit message: initial
Parts:
- added C30: 1n, Capacitor_SMD:C_0402_1005Metric, symbol Device:C
- added C5: 1u, Capacitor_SMD:C_0402_1005Metric, symbol Device:C
- added J1, J2, J3: Conn_02x10_Odd_Even, X3.0CH-Library:Hanxia_HX_PM1.0-2x10P_ZC, symbol Connector_Generic:Conn_02x10_Odd_Even
- added JP1: VREF->3V3, Jumper:SolderJumper-2_P1.3mm_Open_RoundedPad1.0x1.5mm, symbol Jumper:SolderJumper_2_Open
- added U3: REF3033AIDBZR, Package_TO_SOT_SMD:SOT-23, symbol Reference_Voltage:ISL21070CIH320Z-TK
- added U4, U5, U7, U8: PESD4USB5U-TTSX, Package_DFN_QFN:Diodes_UDFN-10_1x2.5mm_P0.5mm, symbol Power_Protection:ESD224DQA
Connections:
- new net +3.3REF: J1.4 (Pin_4), JP1.1 (A), U3.2 (Vout)
- new net +3.3V: J1.3 (Pin_3), JP1.2 (B)
- new net +5V: C5.1, J1.1 (Pin_1), U3.1 (Vin)
- new net CURR1-FILTERED: J2.13 (Pin_13)
- new net CURR2-FILTERED: J2.3 (Pin_3)
- new net CURR3-FILTERED: J1.13 (Pin_13)
- new net ESP-RX: J3.20 (Pin_20), U5.4, U5.7
- new net ESP-TX: J3.19 (Pin_19), U5.2, U5.9
- new net GND: C30.2, C5.2, J1.10 (Pin_10), J1.12 (Pin_12), J1.14 (Pin_14), J1.16 (Pin_16), J1.18 (Pin_18), J1.2 (Pin_2), J1.20 (Pin_20), J2.10 (Pin_10), J2.12 (Pin_12), J2.14 (Pin_14), J2.16 (Pin_16), J2.2 (Pin_2), J2.4 (Pin_4), J2.6 (Pin_6), J2.8 (Pin_8), J3.10 (Pin_10), J3.18 (Pin_18), J3.4 (Pin_4), J3.7 (Pin_7), U3.3 (GND), U4.3 (VSS), U4.8 (VSS), U5.3 (VSS), U5.8 (VSS), U7.3 (VSS), U7.8 (VSS), U8.3 (VSS), U8.8 (VSS)
- new net H1: J2.9 (Pin_9)
- new net H2: J1.19 (Pin_19)
- new net H3: J1.9 (Pin_9)
- new net HALL1-IN: J3.9 (Pin_9), U8.1, U8.10
- new net HALL2-IN: J3.11 (Pin_11), U8.2, U8.9
- new net HALL3-IN: J3.13 (Pin_13), U8.4, U8.7
- new net I2C2-SCL/USART3-TX: J3.8 (Pin_8), U7.1, U7.10
- new net I2C2-SDA/USART3-RX: J3.6 (Pin_6), U7.2, U7.9
- new net IN-CANH: J3.16 (Pin_16)
- new net IN-CANL: J3.14 (Pin_14)
- new net IN-V: C30.1, J1.8 (Pin_8)
- new net L1: J2.11 (Pin_11)
- new net L2: J2.1 (Pin_1)
- new net L3: J1.11 (Pin_11)
- new net MOSTEMP1: J2.7 (Pin_7)
- new net MOSTEMP2: J1.17 (Pin_17)
- new net MOSTEMP3: J1.7 (Pin_7)
- new net NRST: J3.17 (Pin_17), U5.1, U5.10
- new net POWER-STAGE-DISABLE: J1.5 (Pin_5)
- new net POWER-STAGE-LOCKOUT: J1.6 (Pin_6)
- new net SERVO: J3.12 (Pin_12), U5.5, U5.6
- new net SPI1-MISO-ADC2: J2.20 (Pin_20), U4.4, U4.7
- new net SPI1-MOSI: J2.18 (Pin_18), U4.5, U4.6
- new net SPI1-NSS: J2.17 (Pin_17), U4.1, U4.10
- new net SPI1-SCK-ADC: J2.19 (Pin_19), U4.2, U4.9
- new net SWCLK: J3.5 (Pin_5), U7.5, U7.6
- new net SWDIO: J3.3 (Pin_3), U7.4, U7.7
- new net TEMPMOTOR-IN: J3.15 (Pin_15), U8.5, U8.6
- new net USBD+: J3.1 (Pin_1)
- new net USBD-: J3.2 (Pin_2)
- new net VSENSE1: J2.15 (Pin_15)
- new net VSENSE2: J2.5 (Pin_5)
- new net VSENSE3: J1.15 (Pin_15)
Other:
- removed sheet Connectors
- removed sheet Power
- sheet CAN ports: added CAN-RX, CAN-TX, IN-CANH, IN-CANL; removed none
- sheet Filters ports: added HALL1, HALL1-IN, HALL2, HALL2-IN, HALL3, HALL3-IN, PHASE-FILTER-ENABLE1, PHASE-FILTER-ENABLE2, PHASE-FILTER-ENABLE3, TEMPMOTOR, TEMPMOTOR-IN, VSENSE1, VSENSE2, VSENSE3; removed none
- sheet IMU ports: added IMU-SCL, IMU-SDA; removed none
- sheet MCU ports: added CAN-RX, CAN-TX, CURR1-FILTERED, CURR2-FILTERED, CURR3-FILTERED, ESP-RX, ESP-TX, H1, H2, H3, HALL1, HALL2, HALL3, I2C2-SCL/USART3-TX, I2C2-SDA/USART3-RX, IMU-SCL, IMU-SDA, IN-V, L1, L2, L3, MOSTEMP1, MOSTEMP2, MOSTEMP3, NRST, PHASE-FILTER-ENABLE1, PHASE-FILTER-ENABLE2, PHASE-FILTER-ENABLE3, POWER-STAGE-DISABLE, POWER-STAGE-LOCKOUT, SERVO, SPI1-MISO-ADC2, SPI1-MOSI, SPI1-NSS, SPI1-SCK-ADC, SWCLK, SWDIO, TEMPMOTOR, USBD+, USBD-, VSENSE1, VSENSE2, VSENSE3; removed none
- note added: "3.3V Voltage Reference"
- note added: "Bridge JP1 only if U3 is not fitted"
- moved on the sheet: H1, H2
