File: MCU.kicad_sch (KiCad schematic)
At the start: 20 parts, among them U6 STM32F405RGT6, Y1 SX2M8.000M20F30TNN

Commit message: full-route
Parts:
- added TP1, TP2, TP3: TestPoint, TestPoint:TestPoint_Pad_D1.0mm, symbol Connector:TestPoint
Connections:
- net RESERVED1: now also TP1.1
- net RESERVED2: now also TP2.1
- net RESERVED3: now also TP3.1

Commit message: initial
Connections:
- net CAN RX renamed CAN-RX
- net CAN TX renamed CAN-TX
- net CURR1 FILTERED renamed CURR1-FILTERED
- net CURR2 FILTERED renamed CURR2-FILTERED
- net CURR3 FILTERED renamed CURR3-FILTERED
- net I2C2 SCL/USART3 TX renamed I2C2-SCL/USART3-TX
- net I2C2 SDA/USART3 RX renamed I2C2-SDA/USART3-RX
- net IMU SCL renamed IMU-SCL
- net IMU SDA renamed IMU-SDA
- net IN V renamed IN-V
- net LED FAULT renamed LED-FAULT
- net LED RUN renamed LED-RUN
- net PHASE FILTER ENABLE1 renamed PHASE-FILTER-ENABLE1
- net PHASE FILTER ENABLE2 renamed PHASE-FILTER-ENABLE2
- net PHASE FILTER ENABLE3 renamed PHASE-FILTER-ENABLE3
- net POWER STAGE DISABLE renamed POWER-STAGE-DISABLE
- net POWER STAGE LOCKOUT renamed POWER-STAGE-LOCKOUT
