File: Power.kicad_sch (KiCad schematic)
At the start: 2 parts, among them U3 REF3033AIDBZR

Commit message: initial
Parts:
- removed C5: 1u, Capacitor_SMD:C_0402_1005Metric, symbol Device:C
- removed U3: REF3033AIDBZR, Package_TO_SOT_SMD:SOT-23, symbol Reference_Voltage:ISL21070CIH320Z-TK
Other:
- note removed: "3.3V Voltage Reference"
